File: src/zxeightyzon.kicad_pcb (KiCad board)
At the start: 2 copper layers, 82.2 x 62 mm, 27 parts, among them J1 I/O-A 01x10, J2 I/O-B 01x10, J3 GAL 01x10, U1 YM2149, U2 GAL22V10

Commit message: kicad 10
Other:
- board text added: "This is an Open Hardware project. Anyone is free to contribute to it under the OpenSource MIT License. https://github.com/Bambelweeny57/ZXEightyZON"
- board text added: "ZXEightyZON rev 1.0 Designed by Bambelweeny57 for Submeson Brain Corporation"
- board text removed: "This is an Open Hardware project. Anyone is free to contribute to it under the OpenSource MIT License. https://github.com/Bambleweeny57/ZXEightyZON"
- board text removed: "ZXEightyZON rev 1.0 Designed by Bambleweeny57 for Submeson Brain Corporation"
